File: igagev2.kicad_pcb (KiCad board)
At the start: 2 copper layers, 4.3 x 6.4 mm, 34 parts, among them J2 2171820001, SW1 SW_Push, U1 RP2350_80QFN, U2 LTC4162IUFD-SSTM-TRPBF, U3 W25Q16JVSS, Y1 ABM8-272-T3

Commit message: adding additional symbols and design
Parts:
- added C1: 10u, Capacitor_SMD:C_0805_2012Metric, F.Cu at (70.5, 89.6)
- added C10: 4.7u, Capacitor_SMD:C_0402_1005Metric, F.Cu at (100.8, 96.7)
- added C11: 100n, Capacitor_SMD:C_0402_1005Metric, F.Cu at (93.4, 90.4)
- added C12: 100n, Capacitor_SMD:C_0402_1005Metric, F.Cu at (86.6, 99.6)
- added C13: 100n, Capacitor_SMD:C_0402_1005Metric, F.Cu at (90.6, 104.0)
- added C14: 100n, Capacitor_SMD:C_0402_1005Metric, F.Cu at (94.4, 90.4)
- added C15: 100n, Capacitor_SMD:C_0402_1005Metric, F.Cu at (95.4, 104.0)
- added C16: 100n, Capacitor_SMD:C_0402_1005Metric, F.Cu at (98.0, 91.8)
- added C17: 100n, Capacitor_SMD:C_0402_1005Metric, F.Cu at (91.0, 91.0)
- added C18: 100n, Capacitor_SMD:C_0402_1005Metric, F.Cu at (100.0, 99.3)
- added C19: 10u, Capacitor_SMD:C_0805_2012Metric, F.Cu at (72.0, 112.4)
- added C2: 100n, Capacitor_SMD:C_0402_1005Metric, F.Cu at (76.8, 101.3)
- added C2: 100n, Capacitor_SMD:C_0402_1005Metric, F.Cu at (139.4, 132.7)
- added C3: 15p, Capacitor_SMD:C_0402_1005Metric, F.Cu at (103.0, 98.9)
- added C3: 15p, Capacitor_SMD:C_0402_1005Metric, F.Cu at (139.4, 134.6)
- added C4: 15p, Capacitor_SMD:C_0402_1005Metric, F.Cu at (139.4, 136.6)
- added C4: 15p, Capacitor_SMD:C_0402_1005Metric, F.Cu at (103.0, 95.9)
- added C5: 10u, Capacitor_SMD:C_0805_2012Metric, F.Cu at (83.0, 88.5)
- added C6: 4.7u, RP2350_60QFN_minimal:C_0402_1005Metric_small_pads, F.Cu at (89.4, 95.5)
- added C7: 4.7u, RP2350_60QFN_minimal:C_0402_1005Metric_small_pads, F.Cu at (88.4, 95.5)
- added C8: 100n, Capacitor_SMD:C_0402_1005Metric, F.Cu at (93.0, 104.0)
- added C9: 4.7u, Capacitor_SMD:C_0402_1005Metric, F.Cu at (88.9, 93.3)
- added H3: MountingHole, MountingHole:MountingHole_2.7mm_M2.5, F.Cu at (105.6, 68.5)
- added H4: MountingHole, MountingHole:MountingHole_2.7mm_M2.5, F.Cu at (77.7, 68.5)
- added J1: 22272021, molex 22272021:CONN_AE-6410-02A_MOL, F.Cu at (78.6, 134.1)
- added J1: USB_B_Micro, Connector_USB:USB_Micro-B_Amphenol_10103594-0001LF_Horizontal, F.Cu at (66.8, 97.5)
- added J2: Conn_02x18_Odd_Even, Connector_PinHeader_2.54mm:PinHeader_2x18_P2.54mm_Vertical, F.Cu at (67.5, 25.4)
- added J3: Conn_02x18_Odd_Even, Connector_PinHeader_2.54mm:PinHeader_2x18_P2.54mm_Vertical, F.Cu at (113.2, 25.4)
- added J3: 22272021, molex 22272021:CONN_AE-6410-02A_MOL, F.Cu at (78.6, 141.5)
- added J4: SM03B-SRSS-TB, Connector_JST:JST_SH_SM03B-SRSS-TB_1x03-1MP_P1.00mm_Horizontal, F.Cu at (106.8, 89.9)
- added J4: SM03B-SRSS-TB, Connector_JST:JST_SH_SM03B-SRSS-TB_1x03-1MP_P1.00mm_Horizontal, F.Cu at (138.3, 142.3)
- added J5: 22272041, molex 22272041:CONN_AE-6410-04A_MOL, F.Cu at (70.8, 134.1)
- added J6: 22272041, molex 22272041:CONN_AE-6410-04A_MOL, F.Cu at (70.8, 141.5)
- added J7: 22272041, molex 22272041:CONN_AE-6410-04A_MOL, F.Cu at (70.8, 149.0)
- added J8: 22272041, molex 22272041:CONN_AE-6410-04A_MOL, F.Cu at (70.8, 156.4)
- added J9: 22272041, molex 22272041:CONN_AE-6410-04A_MOL, F.Cu at (70.8, 163.9)
- added L1: 3.3u, RP2350_60QFN_minimal:L_pol_2016, F.Cu at (86.8, 95.5)
- added R1: DNF, Resistor_SMD:R_0402_1005Metric, F.Cu at (76.2, 104.5)
- added R1: DNF, Resistor_SMD:R_0402_1005Metric, F.Cu at (126.2, 132.7)
- added R10: 0, Resistor_SMD:R_0402_1005Metric, F.Cu at (76.7, 108.6)
- added R10: 0, Resistor_SMD:R_0402_1005Metric, F.Cu at (126.2, 142.6)
- added R2: 1k, Resistor_SMD:R_0402_1005Metric, F.Cu at (126.2, 134.7)
- added R2: 1k, Resistor_SMD:R_0402_1005Metric, F.Cu at (100.9, 97.9)
- added R4: 1k, Resistor_SMD:R_0402_1005Metric, F.Cu at (126.2, 136.7)
- added R4: 1k, Resistor_SMD:R_0402_1005Metric, F.Cu at (103.1, 82.1)
- added R5: 33, Resistor_SMD:R_0402_1005Metric, F.Cu at (87.1, 93.3)
- added R6: 1k, Resistor_SMD:R_0402_1005Metric, F.Cu at (75.3, 108.6)
- added R6: 1k, Resistor_SMD:R_0402_1005Metric, F.Cu at (126.2, 138.7)
- added R7: 27, Resistor_SMD:R_0402_1005Metric, F.Cu at (86.6, 98.6)
- added R8: 27, Resistor_SMD:R_0402_1005Metric, F.Cu at (86.6, 97.6)
- added R9: DNF, Resistor_SMD:R_0402_1005Metric, F.Cu at (126.2, 140.6)
- added R9: DNF, Resistor_SMD:R_0402_1005Metric, F.Cu at (76.2, 106.2)
- added REF**: SAMTEC_SS4-10-3.00-X-D-K-TR, SS4-10-3.00-L-D-K-TR:SAMTEC_SS4-10-3.00-X-D-K-TR, F.Cu at (175.6, 116.1)
- added SW1: SW_Push, Button_Switch_SMD:SW_Push_1P1T_NO_Vertical_Wuerth_434133025816, F.Cu at (131.0, 140.8)
- added SW1: SW_Push, Button_Switch_SMD:SW_Push_1P1T_NO_Vertical_Wuerth_434133025816, F.Cu at (69.2, 106.3)
- added SW2: SW_Push, Button_Switch_SMD:SW_Push_1P1T_NO_Vertical_Wuerth_434133025816, F.Cu at (101.4, 85.7)
- added SW2: SW_Push, Button_Switch_SMD:SW_Push_1P1T_NO_Vertical_Wuerth_434133025816, F.Cu at (131.0, 145.6)
- added U1: RP2350_60QFN, RP2350_60QFN_minimal:RP2350-QFN-60-1EP_7x7_P0.4mm_EP3.4x3.4mm_ThermalVias, F.Cu at (94.0, 97.5)
- added U2: NCP1117-3.3_SOT223, Package_TO_SOT_SMD:SOT-223-3_TabPin2, F.Cu at (76.8, 89.5)
- added U3: W25Q128JVS, Package_SO:SOIC-8_5.23x5.23mm_P1.27mm, F.Cu at (81.2, 104.5)
- added U3: W25Q128JVS, Package_SO:SOIC-8_5.23x5.23mm_P1.27mm, F.Cu at (132.8, 135.1)
- added Y1: ABM8-272-T3, Crystal:Crystal_SMD_3225-4Pin_3.2x2.5mm, F.Cu at (137.0, 148.3)
- added Y1: ABM8-272-T3, Crystal:Crystal_SMD_3225-4Pin_3.2x2.5mm, F.Cu at (106.4, 97.5)
- moved C21 53.5 mm to (202.4, 67.0)
- moved R5 53.5 mm to (201.1, 54.4)
- moved C10 53.5 mm to (196.0, 70.4)
- moved C11 53.5 mm to (202.6, 62.5)
- moved C12 53.5 mm to (188.7, 65.0)
- moved C13 53.5 mm to (193.7, 54.9)
- moved C14 53.5 mm to (202.3, 59.4)
- moved C15 53.5 mm to (194.7, 54.9)
- moved C16 53.5 mm to (192.9, 70.3)
- moved C17 53.5 mm to (188.5, 61.0)
- moved C18 53.5 mm to (202.6, 63.4)
- moved C2 53.5 mm to (191.6, 46.7)
- moved C20 53.5 mm to (189.4, 56.9)
- moved C6 53.5 mm to (198.6, 57.0)
- moved C8 53.5 mm to (188.3, 63.0)
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- renumbered R3 to R5
Connections:
- C10 pad 1: /1.1V -> +1V1
- C11 pad 1: /1.1V -> +1V1
- C12 pad 1: Net-(U1-QSPI_IOVDD) -> +3V3
- C13 pad 1: Net-(U1-QSPI_IOVDD) -> +3V3
- C14 pad 1: Net-(U1-QSPI_IOVDD) -> +3V3
- C15 pad 1: Net-(U1-QSPI_IOVDD) -> +3V3
- C16 pad 1: Net-(U1-QSPI_IOVDD) -> +3V3
- C17 pad 1: Net-(U1-QSPI_IOVDD) -> +3V3
- C18 pad 1: Net-(U1-QSPI_IOVDD) -> +3V3
- C6 pad 1: /3.3V -> +3V3
- C8 pad 1: /1.1V -> +1V1
- R5 pad 1: /3.3V -> +3V3
Routing:
- net (no net): track 0.00 -> 1013.1 mm, vias 0 -> 13
- net GND: track 28.9 -> 66.4 mm, vias 16 -> 43
- net Net-(U1-USB_DP): track 3.46 -> 7.56 mm
- net Net-(U1-USB_DM): track 3.24 -> 7.10 mm
- net VBUS: track 0.00 -> 2.11 mm
- added copper zone on F.Cu, net (none)
- added copper zone on F.Cu, net GND
- added copper zone on F.Cu, net VBUS
Other:
- board size 4.3 x 6.4 mm -> 105.8 x 97.6 mm
- board text added: "3V3"
- board text added: "ADC 26-29"
- board text added: "BOOTSEL"
- board text added: "DEBUG"
- board text added: "GND"
- board text added: "GP0"
- board text added: "GP1"
- board text added: "GP10"
- board text added: "GP11"
- board text added: "GP12"
- board text added: "GP13"
- board text added: "GP14"
- board text added: "GP15"
- board text added: "GP16"
- board text added: "GP17"
- board text added: "GP18"
- board text added: "GP19"
- board text added: "GP2"
- board text added: "GP20"
- board text added: "GP21"
- board text added: "GP22"
- board text added: "GP23"
- board text added: "GP24"
- board text added: "GP25"
- board text added: "GP26"
- board text added: "GP27"
- board text added: "GP28"
- board text added: "GP29"
- board text added: "GP3"
- board text added: "GP4"
- board text added: "GP5"
- board text added: "GP6"
- board text added: "GP7"
- board text added: "GP8"
- board text added: "GP9"
- board text added: "Minimal Design Example REV3"
- board text added: "Outer Row GND"
- board text added: "RUN"
- board text added: "SWCLK"
- board text added: "SWD"

Commit message: aupdated layout
Parts:
- removed the C2 at (191.6, 46.7)
- removed C20, C21: 100n, Capacitor_SMD:C_0402_1005Metric
- removed the C3 at (191.9, 73.7)
- removed the C4 at (197.4, 73.7)
- removed the C6 at (198.6, 57.0)
- removed the C7 at (198.5, 55.9)
- removed the C9 at (201.1, 56.5)
- removed the L1 at (198.5, 54.2)
- removed the R1 at (183.8, 44.2)
- removed the R10 at (182.8, 47.2)
- removed the R6 at (182.8, 46.2)
- removed the R9 at (182.8, 45.2)
- removed the SW1 at (185.5, 39.4)
- removed the U1 at (94.0, 97.5)
- removed the U1 at (195.4, 63.2)
- removed the U3 at (187.5, 51.1)
- removed the U3 at (81.2, 104.5)
- removed the Y1 at (194.8, 73.8)
- added U1: RP2350_60QFN, rp2350a:RP2350-QFN-60-1EP_7x7_P0.4mm_EP3.4x3.4mm_ThermalVias, F.Cu at (94.0, 97.5)
- moved R100 64.6 mm to (147.9, 69.8)
- moved U3 59.9 mm to (81.2, 104.6), turned to 90 degrees
- moved R101 57.7 mm to (147.9, 71.8), turned to 0 degrees
- moved J3 56.5 mm to (50.1, 92.8), turned to -90 degrees
- moved J1 55.9 mm to (50.2, 86.0), turned to -90 degrees
- moved R5 54.0 mm to (147.9, 63.8), turned to 0 degrees
- moved C11 52.0 mm to (150.8, 67.7)
- moved U2 51.5 mm to (158.3, 66.5)
- moved R8 50.4 mm to (147.9, 67.8), turned to 0 degrees
- moved J2 50.0 mm to (154.0, 59.3), turned to 0 degrees
- moved C18 49.6 mm to (153.7, 71.7)
- moved R7 48.9 mm to (147.9, 65.8), turned to 0 degrees
- moved C14 48.8 mm to (153.7, 63.8)
- moved C13 46.1 mm to (150.8, 71.7), turned to 0 degrees
- moved C10 45.5 mm to (150.8, 65.8), turned to 0 degrees
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Routing:
- net (no net): track 1013.1 -> 444.0 mm, vias 13 -> 5
- net GND: track 66.4 -> 37.5 mm, vias 43 -> 27
- net +3V3: track 0.00 -> 28.4 mm
- net /GPIO0: track 0.00 -> 28.3 mm, vias 0 -> 2
- net Net-(J2-DP1): track 27.7 -> 0.00 mm, vias 2 -> 0
- net Net-(U1-QSPI_IOVDD): track 25.4 -> 0.00 mm
- net GPI00: track 22.4 -> 0.00 mm
- net Net-(J2-DN1): track 21.5 -> 0.00 mm
- net unconnected-(U1-GPIO1-Pad3): track 0.00 -> 20.5 mm
- net unconnected-(U1-GPIO29_ADC3-Pad43): track 0.00 -> 20.3 mm
- net unconnected-(U1-GPIO2-Pad4): track 0.00 -> 20.3 mm
- net unconnected-(U1-GPIO25-Pad37): track 0.00 -> 20.1 mm
- net unconnected-(U1-GPIO28_ADC2-Pad42): track 0.00 -> 20.1 mm
- net unconnected-(U1-GPIO3-Pad5): track 0.00 -> 20.0 mm
- net unconnected-(U1-GPIO4-Pad7): track 0.00 -> 19.9 mm
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