File: igagev2.kicad_sch (KiCad schematic)
At the start: 34 parts, among them J2 2171820001, SW1 SW_Push, U1 RP2350_80QFN, U2 LTC4162IUFD-SSTM-TRPBF, U3 W25Q16JVSS, Y1 ABM8-272-T3

Commit message: adding additional symbols and design
Parts:
- removed C20, C21: 100n, Capacitor_SMD:C_0402_1005Metric, symbol Device:C
- removed R9: DNF, Resistor_SMD:R_0402_1005Metric, symbol Device:R
- removed U1: RP2350_80QFN, RP2350_80QFN_minimal:RP2350-QFN-80-1EP_10x10_P0.4mm_EP3.4x3.4mm_ThermalVias, symbol MCU_RaspberryPi_RP2350:RP2350_80QFN
- removed U3: W25Q16JVSS, Package_SO:SOIC-8_5.23x5.23mm_P1.27mm, symbol Memory_Flash:W25Q16JVSS
- removed Y1: ABM8-272-T3, ABM8-272-T3_ABR, symbol 2024-08-12_02-55-25:ABM8-272-T3
- added J4: SM03B-SRSS-TB, Connector_JST:JST_SH_SM03B-SRSS-TB_1x03-1MP_P1.00mm_Horizontal, symbol Connector_Generic_MountingPin:Conn_01x03_MountingPin
- added R2, R9: 1k, Resistor_SMD:R_0402_1005Metric, symbol Device:R
- added R9: DNF, Resistor_SMD:R_0402_1005Metric, symbol Device:R
- added SW2: SW_Push, Button_Switch_SMD:SW_Push_1P1T_NO_Vertical_Wuerth_434133025816, symbol Switch:SW_Push
- added U1: RP2350_60QFN, RP2350_60QFN_minimal:RP2350-QFN-60-1EP_7x7_P0.4mm_EP3.4x3.4mm_ThermalVias, symbol RP2350-QFN60:RP2350_60QFN
- added U3: W25Q128JVS, Package_SO:SOIC-8_5.23x5.23mm_P1.27mm, symbol Memory_Flash:W25Q128JVS
- added Y1: ABM8-272-T3, Crystal:Crystal_SMD_3225-4Pin_3.2x2.5mm, symbol Device:Crystal_GND24
- renumbered R3 to R5
Connections:
- net GND: now also J4.2 (Pin_2), J4.MP (MountPin), R9.2, U1.47 (VREG_PGND), U1.61 (GND), U3.4 (GND), Y1.2, Y1.4
- net +3V3: now reaches C12.1, C13.1, C14.1, C15.1, C16.1, C17.1, C18.1
- net +3V3: now also C2.1, C6.1, R1.1, R5.1, U1.1 (IOVDD), U1.11 (IOVDD), U1.20 (IOVDD), U1.30 (IOVDD), U1.38 (IOVDD), U1.44 (ADC_AVDD), U1.45 (IOVDD), U1.49 (VREG_VIN), U1.53 (USB_OTP_VDD), U1.54 (QSPI_IOVDD), U3.8 (VCC)
- net XIN: now reaches C3.1
- net XIN: now also U1.21 (XIN), Y1.1
- net at C7.1, L1.1: now also U1.50 (VREG_FB)
- net at C9.1, R5.2: now also U1.46 (VREG_AVDD)
- net at R8.1: now also U1.51 (USB_DM)
- net at C4.1: now also R2.2, Y1.3
- net QSPI_SS: now reaches R10.1
- net QSPI_SS: no longer R6.2
- net FLASH_SS: now reaches R10.2
- net FLASH_SS: now also R1.2, R9.2, U3.1 (~{CS}); no longer R1.1
- net at L1.2: now also U1.48 (VREG_LX)
- net at R6.1: now also U1.60 (QSPI_SS); no longer SW1.2
- net at R7.1: now also U1.52 (USB_DP)
- net 1.1V renamed +1V1
- net +1V1: now also U1.23 (DVDD), U1.39 (DVDD), U1.6 (DVDD)
- removed net 3.3V: C2.1, C6.1, R1.2, R5.1
- new net: R9.1, SW2.1
- new net GPIO0: R9.1, U1.2 (GPIO0)
- new net QSPI_SCLK: U3.6 (CLK)
- new net QSPI_SD0: U1.57 (QSPI_SD0), U3.5 (DI(IO0))
- new net QSPI_SD1: U1.59 (QSPI_SD1), U3.2 (DO(IO1))
- new net QSPI_SD2: U1.58 (QSPI_SD2), U3.3 (IO2)
- new net QSPI_SD3: U1.55 (QSPI_SD3), U3.7 (IO3)
- new net RUN: SW2.2, U1.26 (RUN)
- new net SWCLK: J4.1 (Pin_1), U1.24 (SWCLK)
- new net SWD: J4.3 (Pin_3), U1.25 (SWD)
- new net XOUT: R2.1, U1.22 (XOUT)
- new net ~{USB_BOOT}: R6.2, SW1.2
Other:
- note added: "12MHz Crystal"
- note added: "Flash"
- note added: "JST Debug Connector"
- moved on the sheet: C10, C11, C12, C13, C14, C15, C16, C17, C18, C6, C7, C8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

Commit message: aupdated layout
Parts:
- added J1, J3: 22272021, CONN_AE-6410-02A_MOL, symbol molex 22272021:22272021
- added J5, J6, J7, J8, J9: 22272041, CONN_AE-6410-04A_MOL, symbol molex 22272041:22272041
- renumbered R9 to R4

Commit message: aupdated
Parts:
- U1: footprint RP2350_60QFN_minimal:RP2350-QFN-60-1EP_7x7_P0.4mm_EP3.4x3.4mm_ThermalVias -> rp2350a:RP2350-QFN-60-1EP_7x7_P0.4mm_EP3.4x3.4mm_ThermalVias
Changed lines of the file:
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@@
 			)
 		)
-		(property "Footprint" "RP2350_60QFN_minimal:RP2350-QFN-60-1EP_7x7_P0.4mm_EP3.4x3.4mm_ThermalVias"
+		(property "Footprint" "rp2350a:RP2350-QFN-60-1EP_7x7_P0.4mm_EP3.4x3.4mm_ThermalVias"
 			(at 163.83 127 0)
 			(effects
